File: PCB/main/chu_main_large.kicad_sch (KiCad schematic)
At the start: 123 parts, among them K1 Conn_01x01_Female, K10 Conn_01x01_Female, K11 Conn_01x01_Female, K12 Conn_01x01_Female, K13 Conn_01x01_Female, K14 Conn_01x01_Female, K15 Conn_01x01_Female, K16 Conn_01x01_Female, K17 Conn_01x01_Female, K18 Conn_01x01_Female, K19 Conn_01x01_Female, K2 Conn_01x01_Female, K20 Conn_01x01_Female, K21 Conn_01x01_Female, K22 Conn_01x01_Female, K23 Conn_01x01_Female, K24 Conn_01x01_Female, K25 Conn_01x01_Female, K26 Conn_01x01_Female, K27 Conn_01x01_Female, K28 Conn_01x01_Female, K29 Conn_01x01_Female, K3 Conn_01x01_Female, K30 Conn_01x01_Female, K31 Conn_01x01_Female, K32 Conn_01x01_Female, K4 Conn_01x01_Female, K5 Conn_01x01_Female, K6 Conn_01x01_Female, K7 Conn_01x01_Female, K8 Conn_01x01_Female, K9 Conn_01x01_Female, SW1 SPST_EVQP4, SW2 SPST_EVQP4, SW3 SPST_EVQP4, U0 ChuAcrylic, U1 PiPico_No_SWD, U2 PCA9548APW, U3 MPR121QR2, U4 MPR121QR2, U5 MPR121QR2, U6 MPR121QR2, X1 GP2Y0E03_REAL, X2 GP2Y0E03_REAL, X3 GP2Y0E03_REAL, X4 GP2Y0E03_REAL, X5 GP2Y0E03_REAL

Commit message: initial fork version
Parts:
- K1: value Conn_01x01_Female -> ChuKeyLarge; footprint chu_main:ChuKey -> chu_main:ChuKeyLarge; symbol Connector:Conn_01x01_Female -> chu_main:ChuKeyLarge
- K10, K18, K26: footprint chu_main:ChuKeyBiasLeft -> chu_main:ChuKeyLarge; symbol Connector:Conn_01x01_Female -> chu_main:ChuKeyLarge
- K11, K12, K13, K14, K15, K16, K19, K2, K20, K21, K22, K23, K24, K27, K28, K29, K3, K30, K31, K32, K4, K5, K6, K7, K8: footprint chu_main:ChuKey -> chu_main:ChuKeyLarge; symbol Connector:Conn_01x01_Female -> chu_main:ChuKeyLarge
- K17, K25, K9: footprint chu_main:ChuKeyBiasRight -> chu_main:ChuKeyLarge; symbol Connector:Conn_01x01_Female -> chu_main:ChuKeyLarge
- R14, R15, R16, R17: footprint (none) -> Resistor_SMD:R_0603_1608Metric_Pad0.98x0.95mm_HandSolder
- U0: footprint chu_main:ChuAcrylic -> chu_main:ChuAcrylicLarge; symbol chu_main:ChuAcrylic -> chu_main:ChuAcrylicLarge
